File: kicads/IOW100Paddle/IOW100Paddle.kicad_pcb (KiCad board)
At the start: 4 copper layers, 83.8 x 167.6 mm, 106 parts, among them J1 CONN_02X23, J4 CONN_01X32, J5 CONN_02X23, J6 CONN_01X02, J7 CONN_01X02, Q1 2N7000, Q10 2N7000, Q11 2N7000, Q12 2N7000, Q13 2N7000, Q14 2N7000, Q15 2N7000, Q16 2N7000, Q17 2N3904, Q18 2N3904, Q19 2N3904, Q2 2N7000, Q20 2N3904, Q21 2N3904, Q22 2N3904, Q23 2N3904, Q24 2N3904, Q25 2N3904, Q26 2N3904, Q27 2N3904, Q28 2N3904, Q29 2N3904, Q3 2N7000, Q30 2N3904, Q31 2N3904, Q32 2N3904, Q33 2N7000, Q34 2N7000, Q35 2N7000, Q36 2N7000, Q37 2N7000, Q38 2N7000, Q39 2N7000, Q4 2N7000, Q40 2N7000, Q41 2N7000, Q42 2N7000, Q43 2N7000, Q44 2N7000, Q45 2N7000, Q46 2N7000, Q47 2N7000, Q48 2N7000, Q49 2N3904, Q5 2N7000, Q50 2N3904, Q51 2N3904, Q52 2N3904, Q53 2N3904, Q54 2N3904, Q55 2N3904, Q56 2N3904, Q57 2N3904, Q58 2N3904, Q59 2N3904, Q6 2N7000, Q60 2N3904, Q61 2N3904, Q62 2N3904, Q63 2N3904, Q64 2N3904, Q7 2N7000, Q8 2N7000, Q9 2N7000

Commit message: update manually generated pcbs to include patches and logo
BACKPLANE 2024-04-17
EIGHT 2024-04-17
IOW100PADDLE 2024-04-25
SPVCTL 2024-04-17
Parts:
- added G***: LOGO, LOGO, F.Cu at (11.4, 12.7)
Other:
- net class 5V removed
- net class Default removed
- rule pad_to_mask_clearance: 0.2 -> 0
- board text added: "IOW100Paddle 2023-04-25"
- board text removed: "IOW100Paddle 2023-08-13"
