File: kicads/eight/eight.kicad_pcb (KiCad board)
At the start: 4 copper layers, 200.7 x 73.7 mm, 110 parts, among them J1 CONN_01X03, J10 CONN_01X03, J11 CONN_01X03, J12 CONN_01X03, J13 CONN_01X03, J14 CONN_01X03, J15 CONN_01X03, J16 CONN_01X03, J17 CONN_01X01, J18 CONN_01X01, J19 CONN_01X01, J2 CONN_01X03, J20 CONN_01X01, J21 CONN_01X01, J22 CONN_01X01, J23 CONN_01X01, J24 CONN_01X01, J3 CONN_01X03, J4 CONN_01X03, J5 CONN_01X03, J6 CONN_01X03, J7 CONN_01X03, J8 CONN_01X03, J9 CONN_01X03, U1 6J6, U2 6J6, U3 6J6, U4 6J6, U5 6J6, U6 6J6, U7 6J6, U8 6J6

Commit message: update manually generated pcbs to include patches and logo
BACKPLANE 2024-04-17
EIGHT 2024-04-17
IOW100PADDLE 2024-04-25
SPVCTL 2024-04-17
Parts:
- added G***: LOGO, LOGO, F.Cu at (164.5, 70.5)
Other:
- net class Default removed
- net class FILMNT removed
- net class POWER removed
- rule pad_to_mask_clearance: 0.2 -> 0
- board text added: "EIGHT-2024-04-17"
- board text removed: "EIGHT-2023-05-27"
