File: kicads/backplane/backplane.kicad_pcb (KiCad board)
At the start: 4 copper layers, 431.8 x 457.2 mm, 90 parts, among them J1 CONN_01X32, J10 CONN_01X32, J11 CONN_01X06, J12 CONN_01X32, J13 CONN_01X06, J14 CONN_01X32, J15 CONN_01X32, J16 CONN_01X06, J17 CONN_01X32, J18 CONN_01X06, J19 CONN_01X32, J2 CONN_01X06, J20 CONN_01X06, J21 CONN_01X32, J22 CONN_01X32, J23 CONN_01X06, J24 CONN_01X32, J25 CONN_01X06, J26 CONN_01X32, J27 CONN_01X06, J28 CONN_01X32, J29 CONN_01X32, J3 CONN_01X32, J30 CONN_01X06, J31 CONN_01X32, J32 CONN_01X06, J33 CONN_01X32, J34 CONN_01X06, J35 CONN_01X32, J36 CONN_01X32, J37 CONN_01X06, J38 CONN_01X32, J39 CONN_01X06, J4 CONN_01X06, J40 CONN_01X32, J41 CONN_01X06, J42 CONN_01X32, J43 CONN_01X32, J44 CONN_01X06, J45 CONN_01X32, J46 CONN_01X06, J47 CONN_01X32, J48 CONN_01X06, J49 CONN_01X32, J5 CONN_01X32, J50 CONN_01X32, J51 CONN_01X06, J52 CONN_01X32, J53 CONN_01X06, J54 CONN_01X32, J55 CONN_01X06, J56 CONN_01X32, J57 CONN_01X32, J58 CONN_01X06, J59 CONN_01X32, J6 CONN_01X06, J60 CONN_01X06, J61 CONN_01X32, J62 CONN_01X06, J63 CONN_01X32, J64 CONN_01X32, J65 CONN_01X06, J66 CONN_01X32, J67 CONN_01X06, J68 CONN_01X32, J69 CONN_01X06, J7 CONN_01X32, J70 CONN_01X32, J71 VFF, J72 VFF, J73 +VPP, J74 -VGG, J75 VCC, J76 VFF, J77 VFF, J78 HOLE, J79 HOLE, J8 CONN_01X32, J80 HOLE, J81 HOLE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

Commit message: update manually generated pcbs to include patches and logo
BACKPLANE 2024-04-17
EIGHT 2024-04-17
IOW100PADDLE 2024-04-25
SPVCTL 2024-04-17
Parts:
- added G***: LOGO, LOGO, F.Cu at (363.2, 444.5)
- added J88: Conn_01x04_Pin, Connector_PinHeader_2.54mm:PinHeader_1x04_P2.54mm_Vertical, B.Cu at (359.4, 336.6)
- added J89: Conn_01x08_Pin, Connector_PinHeader_2.54mm:PinHeader_1x08_P2.54mm_Vertical, B.Cu at (359.4, 241.3)
Connections:
- net Net-(J14-Pad4) renamed /clok2
- net Net-(J14-Pad5) renamed /fetch2q
Routing:
- net GND: track 136.1 -> 423.1 mm
- net (no net): track 287.0 -> 0.00 mm
- net /VF5: track 1137.0 -> 1406.2 mm
- net /VF6: track 1092.8 -> 1341.3 mm
- net /VF8: track 1086.4 -> 1325.1 mm
- net /VF7: track 1086.4 -> 1320.5 mm
- net /VF1: track 1086.5 -> 1217.3 mm
- net /VF2: track 1086.5 -> 1216.7 mm
- net /VF4: track 1086.5 -> 1206.7 mm
- net /VF3: track 1086.5 -> 1198.1 mm
- net /VCC: track 4023.3 -> 4132.4 mm
- net /fetch2q: track 400.1 -> 433.1 mm
- net /clok2: track 400.1 -> 430.1 mm
Other:
- net class Default removed
- net class FILAMT removed
- net class POWER removed
- rule pad_to_mask_clearance: 0.2 -> 0
- board text added: "2024-04-17"
- board text added: "ACL"
- board text removed: "2023-08-21"
- board text removed: "AC"

Commit message: fix backplane shorted VPP connector by ground pad
protection diode cathode was shorted to ground

also turn filament connectors 90 degrees for easier wiring
Parts:
- added G***: LOGO, LOGO, B.Cu at (363.2, 444.5)
- moved D2 142.2 mm to (135.9, 238.8)
- moved D3 133.7 mm to (86.4, 228.9), turned to 90 degrees
- moved D1 48.3 mm to (127.0, 215.9), turned to -90 degrees
- moved J72 9.69 mm to (302.9, 120.7), turned to 0 degrees
- moved J77 9.69 mm to (302.9, 336.6), turned to 0 degrees
- moved J71 5.43 mm to (125.1, 120.7), turned to 0 degrees
- moved J76 5.43 mm to (125.1, 336.6), turned to 0 degrees
Routing:
- net /VF1: track 1217.3 -> 1245.0 mm
- net /VF6: track 1341.3 -> 1364.8 mm
- net /VF2: track 1216.7 -> 1239.7 mm
- net /VF4: track 1206.7 -> 1222.7 mm
- net /VF5: track 1406.2 -> 1421.2 mm
- net /VF8: track 1325.1 -> 1336.9 mm
- net /VPP: track 815.3 -> 825.5 mm
- net /VF7: track 1320.5 -> 1329.1 mm
- net /VF3: track 1198.1 -> 1205.3 mm
- net /VCC: track 4132.4 -> 4138.8 mm
- net GND: track 423.1 -> 417.7 mm
Other:
- board text added: "2025-11-29"
- board text removed: "2024-04-17"
